File: CAD/SAO_AMAMW/SAO_AMAMW.kicad_pcb (KiCad board)
At the start: 2 copper layers, 55.3 x 71.6 mm, 28 parts, among them J1 Badgelife_sao_connector_v169b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, U1 TPS61023

Commit message: Production updates
Parts:
- moved R2 7.24 mm to (126.3, 93.6), turned to 0 degrees
Routing:
- net Net-(D2-K): track 5.04 -> 5.67 mm
Changed lines of the file:
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@@
 			(plot_on_all_layers_selection 0x0000000_00000000)
 			(disableapertmacros no)
-			(usegerberextensions no)
-			(usegerberattributes yes)
-			(usegerberadvancedattributes yes)
+			(usegerberextensions yes)
+			(usegerberattributes no)
+			(usegerberadvancedattributes no)
 			(creategerberjobfile no)
 			(dashed_line_dash_ratio 12.000000)
@@
 			(sketchpadsonfab no)
 			(subtractmaskfromsilk yes)
-			(outputformat 4)
+			(outputformat 1)
 			(mirror no)
 			(drillshape 0)
@@
 		(tags "capacitor handsolder")
 		(property "Reference" "C1"
-			(at -1.651 -9.525 180)
+			(at 0.6858 1.8796 180)
 			(layer "B.SilkS")
 			(effects
@@
 		(tags "capacitor handsolder")
 		(property "Reference" "C3"
-			(at -3 0 90)
+			(at -2.8956 -0.3092 90)
 			(layer "B.SilkS")
 			(effects
@@
 		(tags "resistor handsolder")
 		(property "Reference" "R9"
-			(at 1.016 8.636 0)
+			(at -2.9464 -0.0508 0)
 			(layer "B.SilkS")
 			(effects
@@
 		(at 122.047 91.694)
 		(property "Reference" "D2"
-			(at 3.429 -0.762 180)
+			(at 3.048 -2.0574 180)
 			(layer "B.SilkS")
 			(effects
@@
 		(tags "capacitor handsolder")
 		(property "Reference" "C5"
-			(at -0.889 -5.715 90)
+			(at -0.0254 1.6764 90)
 			(layer "B.SilkS")
 			(effects
@@
 	(footprint "Resistor_SMD:R_0805_2012Metric_Pad1.20x1.40mm_HandSolder"
 		(layer "B.Cu")
-		(at 119.253 95.25 -78)
+		(at 126.3142 93.6498)
 		(descr "Resistor SMD 0805 (2012 Metric), square (rectangular) end terminal, IPC_7351 nominal with elongated pad for handsoldering. (Body size source: IPC-SM-782 page 72, https://www.pcb-3d.com/wordpress/wp-content/uploads/ipc-sm-782a_amendment_1_and_2.pdf), generated with kicad-footprint-generator")
 		(tags "resistor handsolder")
 		(property "Reference" "R2"
-			(at -2.819958 0.439297 12)
+			(at -0.1778 -1.9558 0)
 			(layer "B.SilkS")
 			(effects
@@
 		)
 		(property "Value" "56"
-			(at 0 -1.65 102)
+			(at 0 -1.65 360)
 			(layer "B.Fab")
 			(effects
@@
 		)
 		(property "Footprint" "Resistor_SMD:R_0805_2012Metric_Pad1.20x1.40mm_HandSolder"
-			(at 0 0 102)
+			(at 0 0 360)
 			(layer "F.Fab")
 			(hide yes)
@@
 		)
 		(property "Datasheet" "https://www.yageo.com/upload/media/product/productsearch/datasheet/rchip/PYu-RC_Group_51_RoHS_L_12.pdf"
-			(at 0 0 102)
+			(at 0 0 360)
 			(layer "F.Fab")
 			(hide yes)
@@
 		)
 		(property "Description" ""
-			(at 0 0 102)
+			(at 0 0 360)
 			(layer "F.Fab")
 			(hide yes)
@@
 		)
 		(property "MFG" "YAGEO"
-			(at 0 0 102)
+			(at 0 0 360)
 			(layer "B.Fab")
 			(hide yes)
@@
 		)
 		(property "MPN" "RC0805JR-0756RL"
-			(at 0 0 102)
+			(at 0 0 360)
 			(layer "B.Fab")
 			(hide yes)
@@
 		)
 		(property "Vendor 1" "LCSC"
-			(at 0 0 102)
+			(at 0 0 360)
 			(layer "B.Fab")
 			(hide yes)
@@
 		)
 		(property "Vendor 2" "DigiKey"
-			(at 0 0 102)
+			(at 0 0 360)
 			(layer "B.Fab")
 			(hide yes)
@@
 		)
 		(property "Vendor PN 1" "C113305"
-			(at 0 0 102)
+			(at 0 0 360)
 			(layer "B.Fab")
 			(hide yes)
@@
 		)
 		(property "Vendor PN 2" "311-56ARCT-ND"
-			(at 0 0 102)
+			(at 0 0 360)
 			(layer "B.Fab")
 			(hide yes)
@@
 		(attr smd)
 		(fp_line
-			(start -0.227064 0.735)
-			(end 0.227064 0.735)
+			(start -0.227064 -0.735)
+			(end 0.227064 -0.735)
 			(stroke
 				(width 0.12)
@@
 		)
 		(fp_line
-			(start -0.227064 -0.735)
-			(end 0.227064 -0.735)
+			(start -0.227064 0.735)
+			(end 0.227064 0.735)
 			(stroke
 				(width 0.12)
@@
 		)
 		(fp_line
-			(start -1.85 0.95)
-			(end 1.85 0.95)
+			(start -1.85 -0.95)
+			(end -1.85 0.95)
 			(stroke
 				(width 0.05)
@@
 		)
 		(fp_line
-			(start 1.85 0.95)
-			(end 1.85 -0.95)
+			(start -1.85 0.95)
+			(end 1.85 0.95)
 			(stroke
 				(width 0.05)
@@
 		)
 		(fp_line
-			(start -1.85 -0.95)
-			(end -1.85 0.95)
+			(start 1.85 -0.95)
+			(end -1.85 -0.95)
 			(stroke
 				(width 0.05)
@@
 		)
 		(fp_line
-			(start 1.85 -0.95)
-			(end -1.85 -0.95)
+			(start 1.85 0.95)
+			(end 1.85 -0.95)
 			(stroke
 				(width 0.05)
@@
 		)
 		(fp_line
-			(start -1 0.625)
-			(end 1 0.625)
+			(start -1 -0.625)
+			(end -1 0.625)
 			(stroke
 				(width 0.1)
@@
 		)
 		(fp_line
-			(start 1 0.625)
-			(end 1 -0.625)
+			(start -1 0.625)
+			(end 1 0.625)
 			(stroke
 				(width 0.1)
@@
 		)
 		(fp_line
-			(start -1 -0.625)
-			(end -1 0.625)
+			(start 1 -0.625)
+			(end -1 -0.625)
 			(stroke
 				(width 0.1)
@@
 		)
 		(fp_line
-			(start 1 -0.625)
-			(end -1 -0.625)
+			(start 1 0.625)
+			(end 1 -0.625)
 			(stroke
 				(width 0.1)
@@
 		)
 		(fp_text user "${REFERENCE}"
-			(at 0 0 102)
+			(at 0 0 360)
 			(layer "B.Fab")
 			(effects
@@
 		)
 		(pad "1" smd roundrect
-			(at -1 0 282)
+			(at -1 0)
 			(size 1.2 1.4)
 			(layers "B.Cu" "B.Paste" "B.Mask")
@@
 		)
 		(pad "2" smd roundrect
-			(at 1 0 282)
+			(at 1 0)
 			(size 1.2 1.4)
 			(layers "B.Cu" "B.Paste" "B.Mask")
@@
 		(tags "capacitor handsolder")
 		(property "Reference" "C2"
-			(at -3 0 90)
+			(at -2.9972 0.0254 90)
 			(layer "B.SilkS")
 			(effects
@@
 		(tags "resistor handsolder")
 		(property "Reference" "R10"
-			(at -1.397 -8.128 180)
+			(at 2.6416 0.1016 180)
 			(layer "B.SilkS")
 			(effects
 				(font
-					(size 1 1)
-					(thickness 0.15)
+					(size 0.5 0.5)
+					(thickness 0.125)
 				)
 				(justify mirror)
@@
 		(layer "B.SilkS")
 	)
+	(gr_circle
+		(center 137.7188 100.076)
+		(end 137.992366 100.076)
+		(stroke
+			(width 0.15)
+			(type solid)
+		)
+		(fill solid)
+		(layer "B.SilkS")
+	)
 	(gr_poly
 		(pts
@@
 	)
 	(segment
-		(start 119.045088 94.271852)
-		(end 118.745 93.971764)
+		(start 121.087 91.694)
+		(end 121.087 92.766)
 		(width 0.25)
 		(layer "B.Cu")
@@
 	)
 	(segment
-		(start 121.087 91.694)
-		(end 118.745 91.694)
+		(start 121.9708 93.6498)
+		(end 125.3142 93.6498)
 		(width 0.25)
 		(layer "B.Cu")
@@
 	)
 	(segment
-		(start 118.745 93.971764)
-		(end 118.745 91.694)
+		(start 121.087 92.766)
+		(end 121.9708 93.6498)
 		(width 0.25)
 		(layer "B.Cu")
@@
 	)
 	(via
+		(at 128.7018 93.7006)
+		(size 0.8)
+		(drill 0.4)
+		(layers "F.Cu" "B.Cu")
+		(net 7)
+	)
+	(via
 		(at 132.588 112.014)
 		(size 0.8)
@@
 	)
 	(via
-		(at 119.634 97.536)
-		(size 0.8)
-		(drill 0.4)
-		(layers "F.Cu" "B.Cu")
-		(net 7)
-	)
-	(via
 		(at 136.017 86.614)
 		(size 0.8)
@@
 	)
 	(segment
+		(start 127.3142 93.6498)
+		(end 128.651 93.6498)
+		(width 0.25)
+		(layer "B.Cu")
+		(net 7)
+	)
+	(segment
 		(start 135.017 95.25)
 		(end 135.017 93.742)
@@
 	)
 	(segment
-		(start 119.460912 96.228148)
-		(end 119.460912 97.362912)
-		(width 0.25)
-		(layer "B.Cu")
-		(net 7)
-	)
-	(segment
 		(start 143.256 99.076)
 		(end 143.256 99.314)
@@
 	)
 	(segment
-		(start 119.460912 97.362912)
-		(end 119.634 97.536)
+		(start 135.017 93.742)
+		(end 135.001 93.726)
 		(width 0.25)
 		(layer "B.Cu")
@@
 	)
 	(segment
-		(start 135.017 93.742)
-		(end 135.001 93.726)
+		(start 139.573 93.4505)
+		(end 139.573 92.202)
 		(width 0.25)
 		(layer "B.Cu")
@@
 	)
 	(segment
-		(start 139.573 93.4505)
-		(end 139.573 92.202)
+		(start 128.651 93.6498)
+		(end 128.7018 93.7006)
 		(width 0.25)
 		(layer "B.Cu")
@@
 		(hatch edge 0.5)
 		(connect_pads thru_hole_only
-			(clearance 0.1524)
+			(clearance 0.2)
 		)
-		(min_thickness 0.1524)
+		(min_thickness 0.2)
 		(filled_areas_thickness no)
 		(fill yes
