File: CAD/SAO_AMAMW/SAO_AMAMW.kicad_sch (KiCad schematic)
At the start: 32 parts, among them J1 Badgelife_sao_connector_v169b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, U1 TPS61023

Commit message: Updates with new SAO footprint
Updated SAO Footprint. Moved LEDs so they all have the same orientation.
Parts:
- removed JP1, JP2, JP3, JP4, JP5, JP7: SolderJumper_2_Open, Jumper:SolderJumper-2_P1.3mm_Open_TrianglePad1.0x1.5mm, symbol Jumper:SolderJumper_2_Open
- X1: footprint BadgePirates:AMAMW -> drawing:AMAMW

Commit message: Updates for fab
Parts:
- J1: MFG Molex -> Cvilux USA; MPN 0878340619 -> CH87062V200; Vendor 1 LCSC -> Digikey; Vendor PN 1 C9136 -> 2987-CH87062V200-ND
Changed lines of the file:
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@@
 			)
 		)
-		(property "Datasheet" "https://tools.molex.com/pdm_docs/sd/878340619_sd.pdf"
+		(property "Datasheet" "https://www.cvilux.com/uploads/spec/100/291/SPCH031.pdf"
 			(at 63.5 43.18 0)
 			(effects
@@
 			)
 		)
-		(property "MFG" "Molex"
+		(property "MFG" "Cvilux USA"
 			(at 58.42 43.18 0)
 			(effects
@@
 			)
 		)
-		(property "MPN" "0878340619"
+		(property "MPN" "CH87062V200"
 			(at 58.42 43.18 0)
 			(effects
@@
 			)
 		)
-		(property "Vendor 1" "LCSC"
+		(property "Vendor 1" "Digikey"
 			(at 58.42 43.18 0)
 			(effects
@@
 			)
 		)
-		(property "Vendor PN 1" "C9136"
+		(property "Vendor PN 1" "2987-CH87062V200-ND"
 			(at 58.42 43.18 0)
 			(effects

Commit message: Updated BOM
Parts:
- C1: MFG Samsung Electro-Mechanics -> CCTC; MPN CL21A106KOQNNNE -> TCC1206X7R106M250HT; Rating X5R -> X7R; Vendor 2 DigiKey -> (none); Vendor PN 1 C1713 -> C5448932; Vendor PN 2 1276-1096-2-ND -> (none); Voltage 16V -> 25V
Changed lines of the file:
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@@
 			)
 		)
-		(property "Datasheet" "https://media.digikey.com/pdf/Data%20Sheets/Samsung%20PDFs/CL21A106KOQNNNE_Spec.pdf"
+		(property "Datasheet" ""
 			(at 147.32 46.99 0)
 			(effects
@@
 			)
 		)
-		(property "Rating" "X5R"
+		(property "Rating" "X7R"
 			(at 150.241 50.8 0)
 			(effects
@@
 			)
 		)
-		(property "Voltage" "16V"
+		(property "Voltage" "25V"
 			(at 150.241 52.57 0)
 			(effects
@@
 			)
 		)
-		(property "MFG" "Samsung Electro-Mechanics"
+		(property "MFG" "CCTC "
 			(at 147.32 46.99 0)
 			(effects
@@
 			)
 		)
-		(property "MPN" "CL21A106KOQNNNE"
+		(property "MPN" "TCC1206X7R106M250HT"
 			(at 147.32 46.99 0)
 			(effects
@@
 			)
 		)
-		(property "Vendor PN 1" "C1713"
+		(property "Vendor PN 1" "C5448932"
 			(at 147.32 46.99 0)
 			(effects
@@
 			)
 		)
-		(property "Vendor 2" "DigiKey"
+		(property "Vendor 2" ""
 			(at 147.32 46.99 0)
 			(effects
@@
 			)
 		)
-		(property "Vendor PN 2" "1276-1096-2-ND"
+		(property "Vendor PN 2" ""
 			(at 147.32 46.99 0)
 			(effects
